Commit message: cartographer two scan version

File: uc_car_v1/urdf/un_car.urdf (robot description, URDF)
Before this commit: robot Un_car, 8 links, 7 joints
Links:
- link back_left_wheel_link: geometry visual mesh filename=package://uc_car_v1/mesh/wheel.stl scale=0.0009 0.0009 0.0009
- link back_right_wheel_link: geometry visual mesh filename=package://uc_car_v1/mesh/wheel.stl scale=0.0009 0.0009 0.0009
- link body_link: geometry visual mesh filename=package://uc_car_v1/mesh/body.stl scale=0.00059 0.00059 0.00059
- link front_left_wheel_link: geometry visual mesh filename=package://uc_car_v1/mesh/wheel.stl scale=0.0009 0.0009 0.0009
- link front_right_wheel_link: geometry visual mesh filename=package://uc_car_v1/mesh/wheel.stl scale=0.0009 0.0009 0.0009
